File: jeep-in-radio-board/jeep-radio.kicad_pcb (KiCad board)
At the start: 2 copper layers, 45 parts, among them J1 Conn_01x03_Male, J2 Conn_01x03_Male, J3 Conn_01x02_Male, Q1 2N7002, Q2 IRLML6402, Q3 IRLML6402, U1 AP1117-50, U2 MCP100-450D, U3 ATmega328PB-AU, U4 MCP2515-EST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

Commit message: ver 1
Parts:
- added J4: Conn_01x02_Male, Connector_PinHeader_2.54mm:PinHeader_2x01_P2.54mm_Vertical, F.Cu at (149.2, 70.5)
- added MH1: MountingHole, MountingHole:MountingHole_3.2mm_M3_DIN965, F.Cu at (116.2, 71.8)
- added MH2: MountingHole, MountingHole:MountingHole_3.2mm_M3_DIN965, F.Cu at (176.5, 71.8)
- added MH3: MountingHole, MountingHole:MountingHole_3.2mm_M3_DIN965, F.Cu at (116.2, 119.4)
- added MH4: MountingHole, MountingHole:MountingHole_3.2mm_M3_DIN965, F.Cu at (176.5, 119.4)
- moved J3 30.4 mm to (123.2, 70.5)
- moved R8 29.6 mm to (127.6, 88.3), turned to 270 degrees
- moved U5 29.3 mm to (123.2, 80.6)
- moved C10 29.0 mm to (123.3, 87.4)
- moved C11 28.8 mm to (127.6, 80.6)
- moved D1 28.7 mm to (151.6, 97.3), turned to 0 degrees
- moved C4 28.2 mm to (164.6, 117.9), turned to 90 degrees
- moved U4 26.6 mm to (121.3, 92.6)
- moved D2 26.0 mm to (124.5, 111.4)
- moved R9 26.0 mm to (119.4, 111.3)
- moved ICSP1 25.9 mm to (124.5, 103.5)
- moved R4 25.2 mm to (130.0, 108.6)
- moved Q1 24.3 mm to (134.0, 108.6)
- moved R12 24.1 mm to (172.1, 107.1), turned to 90 degrees
- moved Q3 24.0 mm to (154.9, 102.4)
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Connections:
- net Net-(C1-Pad1) renamed /PWR_9
- net Net-(C2-Pad1) renamed /PWR_9_1
- net Net-(D5-Pad1) renamed /VBAT
- U3 pad 23: /BT_ON -> Net-(U3-Pad23)
- U3 pad 25: Net-(U3-Pad25) -> /BT_LED
- U3 pad 26: /BT_LED -> /BT_ON
- U3 pad 29: Net-(U3-Pad29) -> /~RESET~
Routing:
- net /PWR: track 0.00 -> 143.9 mm, vias 0 -> 2
- net /~RESET~: track 0.00 -> 58.5 mm, vias 0 -> 3
- net /VBAT: track 0.00 -> 35.8 mm, vias 0 -> 2
- net /MOSI: track 0.00 -> 34.2 mm, vias 0 -> 2
- net /MISO: track 0.00 -> 25.7 mm
- net /SCK: track 0.00 -> 24.9 mm, vias 0 -> 1
- net /MCP_CLK: track 0.00 -> 24.0 mm, vias 0 -> 2
- net /RXD: track 0.00 -> 21.0 mm
- net GND: track 0.00 -> 20.8 mm, vias 0 -> 37
- net /PWR_9: track 0.00 -> 20.1 mm
- net /TXD: track 0.00 -> 19.1 mm
- net /BT_TX: track 0.00 -> 16.7 mm
- net /XTAL2: track 0.00 -> 16.1 mm
- net /XTAL1: track 0.00 -> 15.9 mm
- net /CAN_CS: track 0.00 -> 13.7 mm
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- added copper zone on B.Cu, net GND
- added copper zone on F.Cu, net GND
Other:
- board outline added: 67.3 x 54 mm
- net class PWR added: clearance 0.3, trace_width 0.6, via_dia 0.8, via_drill 0.4

Commit message: ver 1.001
Parts:
- moved C12 1.05 mm to (163.8, 74.3), turned to 90 degrees
Routing:
- net /AUX_M: track 4.10 -> 2.87 mm
- net Net-(C12-Pad1): track 6.38 -> 7.39 mm
Other:
- board text added: "*"
- board text added: "+9V"
- board text added: "AUX"
- board text added: "CAN"
- board text added: "EN"
- board text added: "H L"
- board text added: "L"
- board text added: "R"
- board text added: "TX RX"
- board text added: "UART"
Changed lines of the file:
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@@
   (general
     (thickness 1.6)
-    (drawings 4)
-    (tracks 305)
+    (drawings 14)
+    (tracks 304)
     (zones 0)
     (modules 50)
@@
     (47 F.CrtYd user)
     (48 B.Fab user)
-    (49 F.Fab user)
+    (49 F.Fab user hide)
   )
   (setup
@@
     (descr "Through hole straight pin header, 2x01, 2.54mm pitch, double rows")
     (tags "Through hole pin header THT 2x01 2.54mm double row")
-    (fp_text reference J4 (at -3.175 0) (layer F.SilkS)
+    (fp_text reference J4 (at 1.27 -3.175) (layer F.SilkS)
       (effects (font (size 1 1) (thickness 0.15)))
     )
@@
     (descr "CP, Radial series, Radial, pin pitch=3.80mm, , diameter=8mm, Electrolytic Capacitor")
     (tags "CP Radial series Radial pin pitch 3.80mm  diameter 8mm Electrolytic Capacitor")
-    (fp_text reference C5 (at 1.9 -5.25 180) (layer F.SilkS)
+    (fp_text reference C5 (at -3.302 -1.778 180) (layer F.SilkS)
       (effects (font (size 1 1) (thickness 0.15)))
     )
@@
     (descr "CP, Radial series, Radial, pin pitch=3.80mm, , diameter=8mm, Electrolytic Capacitor")
     (tags "CP Radial series Radial pin pitch 3.80mm  diameter 8mm Electrolytic Capacitor")
-    (fp_text reference C1 (at 1.9 -5.25 270) (layer F.SilkS)
+    (fp_text reference C1 (at 4.953 -4.572) (layer F.SilkS)
       (effects (font (size 1 1) (thickness 0.15)))
     )
@@
     (tags capacitor)
     (attr smd)
-    (fp_text reference C3 (at 0 -1.65 90) (layer F.SilkS)
+    (fp_text reference C3 (at -2.921 0 180) (layer F.SilkS)
       (effects (font (size 1 1) (thickness 0.15)))
     )
@@
   )
   (module Capacitor_SMD:C_0805_2012Metric (layer F.Cu)
-    (at 164.846 74.549 180)
+    (at 163.83 74.295 90)
     (descr "Capacitor SMD 0805 (2012 Metric), square (rectangular) end terminal, IPC_7351 nominal, (Body size source: https://docs.google.com/spreadsheets/d/1BsfQQcO9C6DZCsRaXUlFlo91Tg2WpOkGARC1WS5S8t0/edit?usp=sharing), generated with kicad-footprint-generator")
     (tags capacitor)
     (attr smd)
-    (fp_text reference C12 (at 2.921 0.254 270) (layer F.SilkS)
-      (effects (font (size 1 1) (thickness 0.15)))
-    )
-    (fp_text value 10uF (at 0 1.65 180) (layer F.Fab)
+    (fp_text reference C12 (at 2.921 0.254 180) (layer F.SilkS)
+      (effects (font (size 1 1) (thickness 0.15)))
+    )
+    (fp_text value 10uF (at 0 1.65 90) (layer F.Fab)
       (effects (font (size 1 1) (thickness 0.15)))
     )
@@
     (fp_line (start 1.68 -0.95) (end 1.68 0.95) (layer F.CrtYd) (width 0.05))
     (fp_line (start 1.68 0.95) (end -1.68 0.95) (layer F.CrtYd) (width 0.05))
-    (fp_text user %R (at 0 0 180) (layer F.Fab)
+    (fp_text user %R (at 0 0 90) (layer F.Fab)
       (effects (font (size 0.5 0.5) (thickness 0.08)))
     )
-    (pad 1 smd roundrect (at -0.9375 0 180) (size 0.975 1.4) (layers F.Cu F.Paste F.Mask) (roundrect_rratio 0.25)
+    (pad 1 smd roundrect (at -0.9375 0 90) (size 0.975 1.4) (layers F.Cu F.Paste F.Mask) (roundrect_rratio 0.25)
       (net 1 "Net-(C12-Pad1)"))
-    (pad 2 smd roundrect (at 0.9375 0 180) (size 0.975 1.4) (layers F.Cu F.Paste F.Mask) (roundrect_rratio 0.25)
+    (pad 2 smd roundrect (at 0.9375 0 90) (size 0.975 1.4) (layers F.Cu F.Paste F.Mask) (roundrect_rratio 0.25)
       (net 71 /AUX_M))
     (model ${KISYS3DMOD}/Capacitor_SMD.3dshapes/C_0805_2012Metric.wrl
@@
     (tags capacitor)
     (attr smd)
-    (fp_text reference C6 (at 0 -1.65 270) (layer F.SilkS)
+    (fp_text reference C6 (at 0 2.54) (layer F.SilkS)
       (effects (font (size 1 1) (thickness 0.15)))
     )
@@
     (tags "capacitor tantalum")
     (attr smd)
-    (fp_text reference C4 (at 0 -1.75 90) (layer F.SilkS)
+    (fp_text reference C4 (at -3.429 0.508 180) (layer F.SilkS)
       (effects (font (size 1 1) (thickness 0.15)))
     )
@@
     (descr "Through hole straight pin header, 1x03, 2.54mm pitch, single row")
     (tags "Through hole pin header THT 1x03 2.54mm single row")
-    (fp_text reference J2 (at 0 8.255) (layer F.SilkS)
+    (fp_text reference J2 (at -3.81 2.54) (layer F.SilkS)
       (effects (font (size 1 1) (thickness 0.15)))
     )
@@
     (descr "Through hole straight pin header, 1x03, 2.54mm pitch, single row")
     (tags "Through hole pin header THT 1x03 2.54mm single row")
-    (fp_text reference J1 (at 0 -2.33 90) (layer F.SilkS)
+    (fp_text reference J1 (at 2.54 1.905 180) (layer F.SilkS)
       (effects (font (size 1 1) (thickness 0.15)))
     )
@@
     (descr "Through hole straight pin header, 2x03, 2.54mm pitch, double rows")
     (tags "Through hole pin header THT 2x03 2.54mm double row")
-    (fp_text reference ICSP1 (at 1.27 -2.33 270) (layer F.SilkS)
+    (fp_text reference ICSP1 (at -3.175 2.54) (layer F.SilkS)
       (effects (font (size 1 1) (thickness 0.15)))
     )
@@
     (tags "Diode MELF ")
     (attr smd)
-    (fp_text reference D4 (at 0 -2.5 180) (layer F.SilkS)
+    (fp_text reference D4 (at 0 2.667 180) (layer F.SilkS)
       (effects (font (size 1 1) (thickness 0.15)))
     )
@@
     (tags "Diode MELF ")
     (attr smd)
-    (fp_text reference D5 (at 0 -2.5 180) (layer F.SilkS)
+    (fp_text reference D5 (at 0.127 2.667 180) (layer F.SilkS)
       (effects (font (size 1 1) (thickness 0.15)))
     )
@@
     (tags diode)
     (attr smd)
-    (fp_text reference D3 (at 0 -1.43 270) (layer F.SilkS)
+    (fp_text reference D3 (at 0 1.905) (layer F.SilkS)
       (effects (font (size 1 1) (thickness 0.15)))
     )
@@
     (tags "CMS SOT")
     (attr smd)
-    (fp_text reference U1 (at 0 -4.5 270) (layer F.SilkS)
+    (fp_text reference U1 (at -1.905 5.08) (layer F.SilkS)
       (effects (font (size 1 1) (thickness 0.15)))
     )
@@
     (tags SOT-23)
     (attr smd)
-    (fp_text reference U2 (at 0 -2.5 270) (layer F.SilkS)
+    (fp_text reference U2 (at -2.54 0) (layer F.SilkS)
       (effects (font (size 1 1) (thickness 0.15)))
     )
@@
     (tags resistor)
     (attr smd)
-    (fp_text reference R12 (at 0 -1.65 90) (layer F.SilkS)
+    (fp_text reference R12 (at 1.016 2.54 180) (layer F.SilkS)
       (effects (font (size 1 1) (thickness 0.15)))
     )
@@
     (tags resistor)
     (attr smd)
-    (fp_text reference R10 (at 0 -1.65 90) (layer F.SilkS)
+    (fp_text reference R10 (at 0.635 -2.54 180) (layer F.SilkS)
       (effects (font (size 1 1) (thickness 0.15)))
     )
@@
     (tags resistor)
     (attr smd)
-    (fp_text reference R6 (at 0 -1.65 180) (layer F.SilkS)
+    (fp_text reference R6 (at 0 1.397 180) (layer F.SilkS)
       (effects (font (size 1 1) (thickness 0.15)))
     )
@@
     (tags resistor)
     (attr smd)
-    (fp_text reference R7 (at 0 -1.65) (layer F.SilkS)
+    (fp_text reference R7 (at -3.175 0.508) (layer F.SilkS)
       (effects (font (size 1 1) (thickness 0.15)))
     )
@@
       (net 22 "Net-(U6-Pad14)"))
   )
+  (gr_text * (at 127 103.505) (layer F.SilkS)
+    (effects (font (size 1.5 1.5) (thickness 0.3)))
+  )
+  (gr_text "H L\n" (at 124.46 73.025) (layer F.SilkS)
+    (effects (font (size 1.5 1.5) (thickness 0.3)))
+  )
+  (gr_text UART (at 144.145 70.485) (layer F.SilkS)
+    (effects (font (size 1.5 1.5) (thickness 0.3)))
+  )
+  (gr_text AUX (at 156.845 70.485) (layer F.SilkS)
+    (effects (font (size 1.5 1.5) (thickness 0.3)))
+  )
+  (gr_text "L\n" (at 166.37 73.66) (layer F.SilkS)
+    (effects (font (size 1.5 1.5) (thickness 0.3)))
+  )
+  (gr_text "R\n" (at 161.29 73.66) (layer F.SilkS)
+    (effects (font (size 1.5 1.5) (thickness 0.3)))
+  )
+  (gr_text "+9V\n" (at 136.525 120.015) (layer F.SilkS)
+    (effects (font (size 1.5 1.5) (thickness 0.3)))
+  )
+  (gr_text EN (at 125.095 120.015) (layer F.SilkS)
+    (effects (font (size 1.5 1.5) (thickness 0.3)))
+  )
+  (gr_text "CAN\n" (at 129.54 70.485) (layer F.SilkS)
+    (effects (font (size 1.5 1.5) (thickness 0.3)))
+  )
+  (gr_text "TX RX\n" (at 150.495 73.66) (layer F.SilkS)
+    (effects (font (size 1.5 1.5) (thickness 0.3)))
+  )
   (gr_line (start 113.03 122.58) (end 113.03 68.58) (layer Edge.Cuts) (width 0.15))
   (gr_line (start 180.34 122.555) (end 113.03 122.58) (layer Edge.Cuts) (width 0.15))
   (gr_line (start 180.34 68.58) (end 180.34 122.515) (layer Edge.Cuts) (width 0.15))
   (gr_line (start 113.03 68.58) (end 180.34 68.58) (layer Edge.Cuts) (width 0.15))
-  (segment (start 169.625 76.28) (end 169.625 78.105) (width 0.25) (layer F.Cu) (net 1))
-  (segment (start 165.7835 74.549) (end 167.894 74.549) (width 0.25) (layer F.Cu) (net 1))
-  (segment (start 167.894 74.549) (end 169.625 76.28) (width 0.25) (layer F.Cu) (net 1))
+  (segment (start 169.625 77.405) (end 169.625 78.105) (width 0.25) (layer F.Cu) (net 1))
+  (segment (start 167.4525 75.2325) (end 169.625 77.405) (width 0.25) (layer F.Cu) (net 1))
+  (segment (start 163.83 75.2325) (end 167.4525 75.2325) (width 0.25) (layer F.Cu) (net 1))
   (via (at 167.005 78.105) (size 0.8) (drill 0.4) (layers F.Cu B.Cu) (net 2))
   (segment (start 165.075 78.105) (end 167.005 78.105) (width 0.25) (layer F.Cu) (net 2))
@@
   (segment (start 159.0825 70.485) (end 157.48 72.0875) (width 0.25) (layer F.Cu) (net 70))
   (segment (start 161.29 70.485) (end 159.0825 70.485) (width 0.25) (layer F.Cu) (net 70))
-  (segment (start 163.83 74.4705) (end 163.9085 74.549) (width 0.25) (layer F.Cu) (net 71))
-  (segment (start 163.83 70.485) (end 163.83 74.4705) (width 0.25) (layer F.Cu) (net 71))
+  (segment (start 163.83 73.3575) (end 163.83 70.485) (width 0.25) (layer F.Cu) (net 71))
   (segment (start 169.8475 70.485) (end 170.18 70.8175) (width 0.25) (layer F.Cu) (net 72))
   (segment (start 166.37 70.485) (end 169.8475 70.485) (width 0.25) (layer F.Cu) (net 72))

Commit message: .
Parts:
- J4: value Conn_01x02_Male -> Conn_01x03_Male; footprint Connector_PinHeader_2.54mm:PinHeader_2x01_P2.54mm_Vertical -> Connector_PinHeader_2.54mm:PinHeader_1x03_P2.54mm_Vertical
- moved C7 13.9 mm to (140.0, 81.4), turned to 180 degrees
- moved U2 12.0 mm to (130.9, 96.0), turned to 90 degrees
- moved D1 8.02 mm to (147.7, 90.3), turned to 90 degrees
- moved R11 8.01 mm to (130.9, 99.8), turned to 180 degrees
- moved R12 6.85 mm to (173.4, 100.3), turned to 180 degrees
- moved C6 6.25 mm to (134.7, 96.1), turned to 90 degrees
- moved C13 5.40 mm to (162.3, 75.4)
- moved C14 3.69 mm to (170.1, 75.4)
- moved R6 3.43 mm to (147.7, 98.4)
- moved R7 3.43 mm to (147.7, 101.0)
- moved Q2 3.42 mm to (143.0, 106.7)
- moved D5 3.28 mm to (167.0, 100.5)
- moved R5 3.27 mm to (138.4, 106.7)
- moved R3 2.90 mm to (127.5, 112.1)
- moved R1 2.84 mm to (131.6, 112.1)
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Connections:
- U3 pad 23: Net-(U3-Pad23) -> /BT_LED
- U3 pad 24: Net-(U3-Pad24) -> /BT_ON
- U3 pad 25: /BT_LED -> Net-(D1-Pad1)
- U3 pad 26: /BT_ON -> Net-(U3-Pad26)
- U3 pad 27: Net-(D1-Pad1) -> /BT_TX
- U3 pad 28: /BT_TX -> Net-(U3-Pad28)
Routing:
- net GND: track 20.8 -> 35.7 mm, vias 37 -> 17
- net /~RESET~: track 58.5 -> 49.4 mm
- net /BT_RX: track 7.22 -> 15.8 mm
- net Net-(D1-Pad1): track 10.6 -> 5.01 mm
- net /BT_ON: track 13.5 -> 7.98 mm
- net /RXD: track 21.0 -> 17.2 mm
- net /VBAT: track 35.8 -> 32.0 mm, vias 2 -> 0
- net Net-(C13-Pad1): track 8.42 -> 4.67 mm
- net /PWR: track 143.9 -> 147.6 mm
- net Net-(C14-Pad1): track 8.66 -> 5.46 mm, vias 2 -> 0
- net ENA_SIG_5V: track 4.14 -> 7.20 mm
- net +9V: track 7.75 -> 10.3 mm
- net /BT_LED: track 6.66 -> 4.20 mm
- net Net-(U4-Pad2): track 12.2 -> 10.2 mm
- net /AUX_L: track 3.95 -> 5.93 mm
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Other:
- net class PWR: clearance 0.3 -> 0.2
- board text added: "(c) github.com/latonita"
- board text added: "EN 9V"
- board text added: "PWR"
- board text added: "R-M-L"
- board text added: "XS-3868"
- board text added: "v 2.0"
- board text removed: "+9V"
- board text removed: "EN"
- board text removed: "L"
- board text removed: "R"
- board text removed: "UART"

Commit message: PCB for xs3868v3
Parts:
- added J5: Conn_01x04_Male, Connector_PinHeader_2.54mm:PinHeader_1x04_P2.54mm_Vertical, F.Cu at (177.5, 103.4)
- added R13: 10k, Resistor_SMD:R_0805_2012Metric, F.Cu at (153.9, 75.1)
- R10: value 1k -> 680
- moved D3 28.5 mm to (156.3, 75.1)
- moved R10 26.6 mm to (158.6, 75.1), turned to 270 degrees
- moved D4 4.83 mm to (154.4, 100.2)
- moved R12 4.83 mm to (168.5, 100.1)
- moved D5 4.83 mm to (162.2, 100.2)
- moved Q3 4.83 mm to (148.1, 100.2)
- moved R6 4.57 mm to (143.1, 98.4)
- moved R7 4.57 mm to (143.1, 101.0)
- moved MH2 0.64 mm to (177.2, 71.8)
- moved MH4 0.64 mm to (177.2, 119.4)
- moved C4 0.64 mm to (163.6, 116.6)
- moved C3 0.63 mm to (159.6, 117.1)
- moved U6 0.44 mm to (149.7, 79.5)
- moved D1 0.20 mm to (147.5, 90.3)
Connections:
- D3 pad 2: /PWR -> /BT_3V3
- D5 pad 1: /VBAT -> /BT_3V3
- R12 pad 2: /VBAT -> /BT_3V3
- U3 pad 23: /BT_LED -> Net-(U3-Pad23)
- U6 pad 10: GND -> Net-(U6-Pad10)
- U6 pad 11: /VBAT -> /BT_3V3
- U6 pad 13: Net-(U6-Pad13) -> /BT_RESET
- U6 pad 18: (no net) -> /BT_TX
- U6 pad 19: /BT_TX -> /BT_RX
- U6 pad 20: /BT_RX -> Net-(U6-Pad20)
- U6 pad 7: Net-(U6-Pad7) -> /BT_LED
- U6 pad 9: Net-(U6-Pad9) -> GND
Routing:
- net /BT_RESET: track 0.00 -> 56.1 mm, vias 0 -> 2
- net /BT_3V3: track 0.00 -> 51.5 mm, vias 0 -> 2
- net /VBAT: track 32.0 -> 0.00 mm
- net /BT_TX: track 17.6 -> 45.5 mm, vias 0 -> 1
- net /BT_RX: track 15.8 -> 41.7 mm, vias 0 -> 1
- net Net-(C14-Pad1): track 5.46 -> 10.7 mm
- net Net-(R13-Pad2): track 0.00 -> 4.39 mm
- net Net-(C12-Pad1): track 6.01 -> 3.54 mm, vias 2 -> 0
- net /BT_ON: track 7.98 -> 6.04 mm
- net Net-(C13-Pad1): track 4.67 -> 4.09 mm
- net Net-(D3-Pad1): track 1.83 -> 2.35 mm
Other:
- board text added: "BT 3V3 RX TX RST"
