File: jeep-in-radio-board/jeep-radio.kicad_pcb (KiCad board)
At the start: 2 copper layers, 67.3 x 54 mm, 52 parts, among them J1 Conn_01x03_Male, J2 Conn_01x03_Male, J3 Conn_01x02_Male, J4 Conn_01x03_Male, J5 Conn_01x04_Male, Q1 2N7002, Q2 IRLML6402, Q3 IRLML6402, U1 AP1117-50, U2 MCP100-450D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

Commit message: pcb fix
Routing:
- net /BT_3V3: track 51.5 -> 49.7 mm
- net Net-(R13-Pad2): track 4.39 -> 5.76 mm
- net /BT_RESET: track 56.1 -> 56.7 mm
Changed lines of the file:
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@@
     (thickness 1.6)
     (drawings 24)
-    (tracks 326)
+    (tracks 332)
     (zones 0)
     (modules 52)
@@
     (tags "Diode MELF ")
     (attr smd)
-    (fp_text reference D4 (at 0 2.667 180) (layer F.SilkS)
+    (fp_text reference D4 (at 0 -2.413 180) (layer F.SilkS)
       (effects (font (size 1 1) (thickness 0.15)))
     )
@@
     (tags "Diode MELF ")
     (attr smd)
-    (fp_text reference D5 (at 0.127 2.667 180) (layer F.SilkS)
+    (fp_text reference D5 (at 0.127 -2.413 180) (layer F.SilkS)
       (effects (font (size 1 1) (thickness 0.15)))
     )
@@
     (tags resistor)
     (attr smd)
-    (fp_text reference R12 (at 0 1.905) (layer F.SilkS)
+    (fp_text reference R12 (at 0.127 -1.778) (layer F.SilkS)
       (effects (font (size 1 1) (thickness 0.15)))
     )
@@
   (gr_line (start 180.34 68.58) (end 180.34 122.515) (layer Edge.Cuts) (width 0.15))
   (gr_line (start 113.03 68.58) (end 180.34 68.58) (layer Edge.Cuts) (width 0.15))
-  (segment (start 166.66 76.7925) (end 166.243 76.3755) (width 0.25) (layer F.Cu) (net 1))
-  (segment (start 166.66 79.74) (end 166.66 76.7925) (width 0.25) (layer F.Cu) (net 1))
-  (segment (start 170.053 76.963) (end 170.053 76.3755) (width 0.25) (layer F.Cu) (net 2))
-  (segment (start 167.767 81.788) (end 170.053 79.502) (width 0.25) (layer F.Cu) (net 2))
-  (segment (start 165.608 81.788) (end 167.767 81.788) (width 0.25) (layer F.Cu) (net 2))
-  (segment (start 165.36 79.74) (end 165.36 81.54) (width 0.25) (layer F.Cu) (net 2))
-  (segment (start 170.053 79.502) (end 170.053 76.963) (width 0.25) (layer F.Cu) (net 2))
-  (segment (start 165.36 81.54) (end 165.608 81.788) (width 0.25) (layer F.Cu) (net 2))
-  (segment (start 162.306 77.216) (end 164.06 78.97) (width 0.25) (layer F.Cu) (net 3))
-  (segment (start 162.306 76.3755) (end 162.306 77.216) (width 0.25) (layer F.Cu) (net 3))
-  (segment (start 164.06 78.97) (end 164.06 79.74) (width 0.25) (layer F.Cu) (net 3))
+  (segment (start 165.76 77.826) (end 165.76 79.64) (width 0.25) (layer F.Cu) (net 1))
+  (segment (start 166.243 76.3755) (end 166.243 77.343) (width 0.25) (layer F.Cu) (net 1))
+  (segment (start 166.243 77.343) (end 165.76 77.826) (width 0.25) (layer F.Cu) (net 1))
+  (segment (start 164.46 80.94) (end 165.054 81.534) (width 0.25) (layer F.Cu) (net 2))
+  (segment (start 164.46 79.64) (end 164.46 80.94) (width 0.25) (layer F.Cu) (net 2))
+  (segment (start 165.054 81.534) (end 166.4335 81.534) (width 0.25) (layer F.Cu) (net 2))
+  (segment (start 170.053 77.9145) (end 170.053 76.3755) (width 0.25) (layer F.Cu) (net 2))
+  (segment (start 166.4335 81.534) (end 170.053 77.9145) (width 0.25) (layer F.Cu) (net 2))
+  (segment (start 162.306 77.2795) (end 162.306 76.3755) (width 0.25) (layer F.Cu) (net 3))
+  (segment (start 163.16 79.64) (end 163.16 78.1335) (width 0.25) (layer F.Cu) (net 3))
+  (segment (start 163.16 78.1335) (end 162.306 77.2795) (width 0.25) (layer F.Cu) (net 3))
   (segment (start 135.225 71.755) (end 135.8125 71.755) (width 0.25) (layer F.Cu) (net 8))
   (segment (start 135.8125 71.755) (end 137.033 71.755) (width 0.25) (layer F.Cu) (net 8))
@@
   (segment (start 147.069 91.065) (end 147.701 91.697) (width 0.25) (layer F.Cu) (net 59))
   (segment (start 143.95 91.065) (end 147.069 91.065) (width 0.25) (layer F.Cu) (net 59))
-  (segment (start 158.86 76.2315) (end 158.623 75.9945) (width 0.25) (layer F.Cu) (net 60))
-  (segment (start 158.86 79.74) (end 158.86 76.2315) (width 0.25) (layer F.Cu) (net 60))
+  (segment (start 158.623 77.1525) (end 158.623 75.9945) (width 0.25) (layer F.Cu) (net 60))
+  (segment (start 157.96 79.64) (end 157.96 77.8155) (width 0.25) (layer F.Cu) (net 60))
+  (segment (start 157.96 77.8155) (end 158.623 77.1525) (width 0.25) (layer F.Cu) (net 60))
   (segment (start 147.32 84.455) (end 147.32 73.025) (width 0.25) (layer F.Cu) (net 61))
   (segment (start 143.95 87.065) (end 144.71 87.065) (width 0.25) (layer F.Cu) (net 61))
@@
   (segment (start 150.4465 106.68) (end 151.7165 107.95) (width 0.6) (layer F.Cu) (net 72))
   (segment (start 144.002 106.68) (end 150.4465 106.68) (width 0.6) (layer F.Cu) (net 72))
-  (segment (start 152.36 77.5585) (end 153.924 75.9945) (width 0.25) (layer F.Cu) (net 75))
-  (segment (start 152.36 79.74) (end 152.36 77.5585) (width 0.25) (layer F.Cu) (net 75))
+  (segment (start 151.46 79.64) (end 151.46 76.632) (width 0.25) (layer F.Cu) (net 75))
+  (segment (start 152.146 75.946) (end 153.924 75.946) (width 0.25) (layer F.Cu) (net 75))
+  (segment (start 151.46 76.632) (end 152.146 75.946) (width 0.25) (layer F.Cu) (net 75))
   (via (at 152.654 93.218) (size 0.8) (drill 0.4) (layers F.Cu B.Cu) (net 79))
   (segment (start 152.76 95.44) (end 152.76 93.324) (width 0.25) (layer F.Cu) (net 79))
   (segment (start 152.76 93.324) (end 152.654 93.218) (width 0.25) (layer F.Cu) (net 79))
-  (via (at 151.384 77.47) (size 0.8) (drill 0.4) (layers F.Cu B.Cu) (net 79))
-  (segment (start 151.384 91.948) (end 151.384 77.47) (width 0.25) (layer B.Cu) (net 79))
-  (segment (start 152.654 93.218) (end 151.384 91.948) (width 0.25) (layer B.Cu) (net 79))
-  (segment (start 152.4485 74.1195) (end 153.924 74.1195) (width 0.25) (layer F.Cu) (net 79))
-  (segment (start 151.384 77.47) (end 151.384 75.184) (width 0.25) (layer F.Cu) (net 79))
-  (segment (start 151.384 75.184) (end 152.4485 74.1195) (width 0.25) (layer F.Cu) (net 79))
   (segment (start 172.72 110.998) (end 177.546 110.998) (width 0.25) (layer B.Cu) (net 79))
   (segment (start 152.654 93.218) (end 154.94 93.218) (width 0.25) (layer B.Cu) (net 79))
   (segment (start 154.94 93.218) (end 172.72 110.998) (width 0.25) (layer B.Cu) (net 79))
+  (segment (start 151.384 91.948) (end 151.384 74.733685) (width 0.25) (layer B.Cu) (net 79))
+  (via (at 151.384 74.168) (size 0.8) (drill 0.4) (layers F.Cu B.Cu) (net 79))
+  (segment (start 152.654 93.218) (end 151.384 91.948) (width 0.25) (layer B.Cu) (net 79))
+  (segment (start 151.384 74.733685) (end 151.384 74.168) (width 0.25) (layer B.Cu) (net 79))
+  (segment (start 153.924 74.1195) (end 151.4325 74.1195) (width 0.25) (layer F.Cu) (net 79))
+  (segment (start 151.4325 74.1195) (end 151.384 74.168) (width 0.25) (layer F.Cu) (net 79))
   (segment (start 164.6275 100.1545) (end 164.579 100.203) (width 0.6) (layer F.Cu) (net 80))
   (segment (start 167.513 100.1545) (end 164.6275 100.1545) (width 0.6) (layer F.Cu) (net 80))
-  (segment (start 164.579 100.203) (end 164.579 97.676) (width 0.6) (layer F.Cu) (net 80))
-  (via (at 164.592 97.663) (size 0.8) (drill 0.4) (layers F.Cu B.Cu) (net 80))
-  (segment (start 164.579 97.676) (end 164.592 97.663) (width 0.6) (layer F.Cu) (net 80))
-  (via (at 153.67 77.724) (size 0.8) (drill 0.4) (layers F.Cu B.Cu) (net 80))
-  (segment (start 153.67 79.73) (end 153.66 79.74) (width 0.6) (layer F.Cu) (net 80))
-  (segment (start 153.67 77.724) (end 153.67 79.73) (width 0.6) (layer F.Cu) (net 80))
-  (segment (start 156.337 77.089) (end 156.337 75.8445) (width 0.6) (layer F.Cu) (net 80))
-  (segment (start 153.67 77.724) (end 155.702 77.724) (width 0.6) (layer F.Cu) (net 80))
-  (segment (start 155.702 77.724) (end 156.337 77.089) (width 0.6) (layer F.Cu) (net 80))
-  (segment (start 153.67 81.603315) (end 153.67 77.724) (width 0.6) (layer B.Cu) (net 80))
-  (segment (start 164.592 97.663) (end 164.592 92.456) (width 0.6) (layer B.Cu) (net 80))
-  (segment (start 164.592 92.456) (end 153.67 81.603315) (width 0.6) (layer B.Cu) (net 80))
-  (segment (start 170.307 103.378) (end 177.546 103.378) (width 0.6) (layer B.Cu) (net 80))
-  (segment (start 164.592 97.663) (end 170.307 103.378) (width 0.6) (layer B.Cu) (net 80))
+  (segment (start 152.76 79.64) (end 152.76 77.554502) (width 0.6) (layer F.Cu) (net 80))
+  (segment (start 152.76 77.554502) (end 152.8445 77.470002) (width 0.6) (layer F.Cu) (net 80))
+  (segment (start 153.410185 77.470002) (end 152.8445 77.470002) (width 0.6) (layer F.Cu) (net 80))
+  (segment (start 155.574998 77.470002) (end 153.410185 77.470002) (width 0.6) (layer F.Cu) (net 80))
+  (segment (start 156.337 75.8445) (end 156.337 76.708) (width 0.6) (layer F.Cu) (net 80))
+  (segment (start 156.337 76.708) (end 155.574998 77.470002) (width 0.6) (layer F.Cu) (net 80))
+  (segment (start 164.579 100.203) (end 164.579 99.603) (width 0.6) (layer F.Cu) (net 80))
+  (via (at 152.908 82.042) (size 0.8) (drill 0.4) (layers F.Cu B.Cu) (net 80))
+  (segment (start 152.76 79.64) (end 152.76 81.894) (width 0.6) (layer F.Cu) (net 80))
+  (segment (start 152.76 81.894) (end 152.908 82.042) (width 0.6) (layer F.Cu) (net 80))
+  (segment (start 167.639968 96.773968) (end 167.64 96.773968) (width 0.6) (layer B.Cu) (net 80))
+  (via (at 167.64 96.773968) (size 0.8) (drill 0.4) (layers F.Cu B.Cu) (net 80))
+  (segment (start 167.5915 96.822468) (end 167.64 96.773968) (width 0.6) (layer F.Cu) (net 80))
+  (segment (start 167.5915 100.076) (end 167.5915 96.822468) (width 0.6) (layer F.Cu) (net 80))
+  (segment (start 152.908 82.042) (end 167.639968 96.773968) (width 0.6) (layer B.Cu) (net 80))
+  (segment (start 174.244032 103.378) (end 168.039999 97.173967) (width 0.6) (layer B.Cu) (net 80))
+  (segment (start 177.546 103.378) (end 174.244032 103.378) (width 0.6) (layer B.Cu) (net 80))
+  (segment (start 168.039999 97.173967) (end 167.64 96.773968) (width 0.6) (layer B.Cu) (net 80))
   (zone (net 0) (net_name "") (layers F&B.Cu) (hatch edge 0.508)
     (connect_pads (clearance 0.508))
