File: jeep-in-radio-board/jeep-radio.sch (KiCad schematic (older format))
At the start: 18 parts, among them Q1 2N7002, Q2 IRLML6402, Q3 IRLML6402, U1 AP1117-50, U2 MCP100-450D

Commit message: schematics 0.1
Parts:
- added C10, C11, C7: 100nF, Capacitor_SMD:C_0805_2012Metric, symbol Device:C
- added C12, C13, C14: 10uF, Capacitor_SMD:C_0805_2012Metric, symbol Device:CP
- added C8, C9: 22pF, Capacitor_SMD:C_0805_2012Metric, symbol Device:C
- added D1: 1N4001, Diode_SMD:D_MELF, symbol Diode:1N4002
- added D2, D3: LED, LED_SMD:LED_0603_1608Metric, symbol Device:LED
- added D4, D5: 1N4001, Diode_SMD:D_MELF, symbol Diode:1N4001
- added ICSP1: Conn_02x03_Odd_Even, Connector_PinHeader_2.54mm:PinHeader_2x03_P2.54mm_Vertical, symbol Connector_Generic:Conn_02x03_Odd_Even
- added J1, J2: Conn_01x03_Male, Connector_PinHeader_2.54mm:PinHeader_1x03_P2.54mm_Vertical, symbol Connector:Conn_01x03_Male
- added J3: Conn_01x02_Male, Connector_PinHeader_2.54mm:PinHeader_2x01_P2.54mm_Vertical, symbol Connector:Conn_01x02_Male
- added R10, R12, R9: 1k, Resistor_SMD:R_0805_2012Metric, symbol Device:R
- added R11, R8: 10k, Resistor_SMD:R_0805_2012Metric, symbol Device:R
- added U3: ATmega328PB-AU, Package_QFP:TQFP-32_7x7mm_P0.8mm, symbol MCU_Microchip_ATmega:ATmega328PB-AU
- added U4: MCP2515-EST, Package_SO:TSSOP-20_4.4x6.5mm_P0.65mm, symbol Interface_CAN_LIN:MCP2515-EST
- added U5: MCP2551-I-SN, Package_SO:SOIC-8_3.9x4.9mm_P1.27mm, symbol Interface_CAN_LIN:MCP2551-I-SN
- added U6: XS3868, latonita:XS3868, symbol latonita-kicad-library:XS3868
- added Y1: Crystal, Crystal:Crystal_SMD_HC49-SD, symbol Device:Crystal
- C1, C5: footprint Capacitor_THT:CP_Radial_D10.0mm_P3.80mm -> Capacitor_THT:CP_Radial_D8.0mm_P3.80mm
- C2, C3, C6: footprint Capacitor_SMD:C_0603_1608Metric -> Capacitor_SMD:C_0805_2012Metric
Connections:
- net labels added: AUX_L, AUX_M, AUX_R, BT_LED, BT_PWR, BT_RX, BT_TX, CAN_CS, CAN_H, CAN_INT, CAN_L, MCP_CLK, MISO, MOSI, RXD, SCK, TXD, XTAL1, XTAL2
- net labels removed: BT_POWER
- wire segments 67 -> 164

Commit message: ver 1
Parts:
- added J4: Conn_01x02_Male, Connector_PinHeader_2.54mm:PinHeader_2x01_P2.54mm_Vertical, symbol Connector:Conn_01x02_Male
- added MH1, MH2, MH3, MH4: MountingHole, MountingHole:MountingHole_3.2mm_M3_DIN965, symbol Mechanical:MountingHole
Connections:
- net labels added: PWR_9, PWR_9_1, VBAT
- wire segments 164 -> 167
Changed lines of the file:
@@
 $EndComp
 Wire Wire Line
-	5600 5650 5950 5650
-Text Label 5750 5650 0    50   ~ 0
+	2700 5650 3050 5650
+Text Label 2850 5650 0    50   ~ 0
 ~RESET~
 $Comp
@@
 	2700 5350 3050 5350
 Text Label 2850 5350 0    50   ~ 0
-BT_LED
+BT_ON
 Wire Wire Line
 	2700 5550 3600 5550
@@
 $EndComp
 Wire Wire Line
-	2700 5050 3050 5050
-Text Label 2850 5050 0    50   ~ 0
-BT_ON
+	2700 5250 3050 5250
+Text Label 2850 5250 0    50   ~ 0
+BT_LED
 $Comp
 L Device:Crystal Y1
@@
 Text Label 10150 1000 0    50   ~ 0
 CAN_L
+$Comp
+L Connector:Conn_01x02_Male J4
+U 1 1 5B97388B
+P 9950 1400
+F 0 "J4" H 9950 1500 50  0000 C CNN
+F 1 "Conn_01x02_Male" H 10056 1487 50  0001 C CNN
+F 2 "Connector_PinHeader_2.54mm:PinHeader_2x01_P2.54mm_Vertical" H 9950 1400 50  0001 C CNN
+F 3 "~" H 9950 1400 50  0001 C CNN
+	1    9950 1400
+	1    0    0    -1
+$EndComp
+Wire Wire Line
+	10150 1400 10350 1400
+Wire Wire Line
+	10150 1500 10350 1500
+Text Label 10150 1400 0    50   ~ 0
+TXD
+Text Label 10150 1500 0    50   ~ 0
+RXD
+$Comp
+L Mechanical:MountingHole MH1
+U 1 1 5B97A4F3
+P 8650 6350
+F 0 "MH1" H 8750 6396 50  0000 L CNN
+F 1 "MountingHole" H 8750 6305 50  0000 L CNN
+F 2 "MountingHole:MountingHole_3.2mm_M3_DIN965" H 8650 6350 50  0001 C CNN
+F 3 "~" H 8650 6350 50  0001 C CNN
+	1    8650 6350
+	1    0    0    -1
+$EndComp
+$Comp
+L Mechanical:MountingHole MH2
+U 1 1 5B98D251
+P 8900 6350
+F 0 "MH2" H 9000 6396 50  0000 L CNN
+F 1 "MountingHole" H 9000 6305 50  0000 L CNN
+F 2 "MountingHole:MountingHole_3.2mm_M3_DIN965" H 8900 6350 50  0001 C CNN
+F 3 "~" H 8900 6350 50  0001 C CNN
+	1    8900 6350
+	1    0    0    -1
+$EndComp
+$Comp
+L Mechanical:MountingHole MH3
+U 1 1 5B98D2C7
+P 9150 6350
+F 0 "MH3" H 9250 6396 50  0000 L CNN
+F 1 "MountingHole" H 9250 6305 50  0000 L CNN
+F 2 "MountingHole:MountingHole_3.2mm_M3_DIN965" H 9150 6350 50  0001 C CNN
+F 3 "~" H 9150 6350 50  0001 C CNN
+	1    9150 6350
+	1    0    0    -1
+$EndComp
+$Comp
+L Mechanical:MountingHole MH4
+U 1 1 5B98D343
+P 9400 6350
+F 0 "MH4" H 9500 6396 50  0000 L CNN
+F 1 "MountingHole" H 9500 6305 50  0000 L CNN
+F 2 "MountingHole:MountingHole_3.2mm_M3_DIN965" H 9400 6350 50  0001 C CNN
+F 3 "~" H 9400 6350 50  0001 C CNN
+	1    9400 6350
+	1    0    0    -1
+$EndComp
+Text Label 2100 1200 0    50   ~ 0
+PWR_9
+Text Label 2900 1900 0    50   ~ 0
+PWR_9_1
+Text Label 9150 5200 0    50   ~ 0
+VBAT
+Text Label 5700 5650 0    50   ~ 0
+~RESET~
+Wire Wire Line
+	5600 5650 5950 5650
 $EndSCHEMATC

Commit message: .
Parts:
- J4: value Conn_01x02_Male -> Conn_01x03_Male; footprint Connector_PinHeader_2.54mm:PinHeader_2x01_P2.54mm_Vertical -> Connector_PinHeader_2.54mm:PinHeader_1x03_P2.54mm_Vertical; symbol Connector:Conn_01x02_Male -> Connector:Conn_01x03_Male
Connections:
- wire segments 167 -> 169
Other:
- moved on the sheet: D1
Changed lines of the file:
@@
 L Diode:1N4002 D1
 U 1 1 5B972DB2
-P 3200 5450
-F 0 "D1" H 3250 5300 50  0000 C CNN
-F 1 "1N4001" H 3250 5200 50  0000 C CNN
-F 2 "Diode_SMD:D_MELF" H 3200 5275 50  0001 C CNN
-F 3 "http://www.vishay.com/docs/88503/1n4001.pdf" H 3200 5450 50  0001 C CNN
-	1    3200 5450
-	1    0    0    -1
-$EndComp
+P 3200 5250
+F 0 "D1" H 3250 5100 50  0000 C CNN
+F 1 "1N4001" H 3250 5000 50  0000 C CNN
+F 2 "Diode_SMD:D_MELF" H 3200 5075 50  0001 C CNN
+F 3 "http://www.vishay.com/docs/88503/1n4001.pdf" H 3200 5250 50  0001 C CNN
+	1    3200 5250
+	1    0    0    -1
+$EndComp
+Text Label 3350 5250 0    50   ~ 0
+BT_RX
+Wire Wire Line
+	2700 5150 3050 5150
+Text Label 2850 5150 0    50   ~ 0
+BT_ON
+Wire Wire Line
+	2700 5450 3600 5450
 Text Label 3350 5450 0    50   ~ 0
-BT_RX
-Wire Wire Line
-	2700 5350 3050 5350
-Text Label 2850 5350 0    50   ~ 0
-BT_ON
-Wire Wire Line
-	2700 5550 3600 5550
-Text Label 3350 5550 0    50   ~ 0
 BT_TX
 Wire Wire Line
@@
 $EndComp
 Wire Wire Line
-	2700 5250 3050 5250
-Text Label 2850 5250 0    50   ~ 0
+	2700 5050 3050 5050
+Text Label 2850 5050 0    50   ~ 0
 BT_LED
 $Comp
@@
 	2700 4150 3800 4150
 Wire Wire Line
-	3050 5450 2700 5450
+	3050 5250 2700 5250
 Wire Wire Line
 	3800 4150 3800 5350
@@
 	3800 5350 4400 5350
 Wire Wire Line
-	3350 5450 3600 5450
+	3350 5250 3600 5250
 $Comp
 L power:GND #PWR05
@@
 P 6100 1000
 F 0 "ICSP1" H 6150 1317 50  0000 C CNN
-F 1 "Conn_02x03_Odd_Even" H 6150 1226 50  0000 C CNN
+F 1 "Conn_02x03_Odd_Even" H 6150 1226 50  0001 C CNN
 F 2 "Connector_PinHeader_2.54mm:PinHeader_2x03_P2.54mm_Vertical" H 6100 1000 50  0001 C CNN
 F 3 "~" H 6100 1000 50  0001 C CNN
@@
 CAN_L
 $Comp
-L Connector:Conn_01x02_Male J4
+L Connector:Conn_01x03_Male J4
 U 1 1 5B97388B
 P 9950 1400
 F 0 "J4" H 9950 1500 50  0000 C CNN
-F 1 "Conn_01x02_Male" H 10056 1487 50  0001 C CNN
-F 2 "Connector_PinHeader_2.54mm:PinHeader_2x01_P2.54mm_Vertical" H 9950 1400 50  0001 C CNN
+F 1 "Conn_01x03_Male" H 10056 1487 50  0001 C CNN
+F 2 "Connector_PinHeader_2.54mm:PinHeader_1x03_P2.54mm_Vertical" H 9950 1400 50  0001 C CNN
 F 3 "~" H 9950 1400 50  0001 C CNN
 	1    9950 1400
@@
 $EndComp
 Wire Wire Line
+	10150 1300 10350 1300
+Wire Wire Line
 	10150 1400 10350 1400
-Wire Wire Line
-	10150 1500 10350 1500
+Text Label 10150 1300 0    50   ~ 0
+TXD
 Text Label 10150 1400 0    50   ~ 0
-TXD
-Text Label 10150 1500 0    50   ~ 0
 RXD
 $Comp
@@
 Wire Wire Line
 	5600 5650 5950 5650
+$Comp
+L power:GND #PWR0104
+U 1 1 5B9BAC5C
+P 10250 1550
+F 0 "#PWR0104" H 10250 1300 50  0001 C CNN
+F 1 "GND" H 10255 1377 50  0000 C CNN
+F 2 "" H 10250 1550 50  0001 C CNN
+F 3 "" H 10250 1550 50  0001 C CNN
+	1    10250 1550
+	1    0    0    -1
+$EndComp
+Wire Wire Line
+	10150 1500 10250 1500
+Wire Wire Line
+	10250 1500 10250 1550
 $EndSCHEMATC

Commit message: PCB for xs3868v3
Parts:
- added J5: Conn_01x04_Male, Connector_PinHeader_2.54mm:PinHeader_1x04_P2.54mm_Vertical, symbol Connector:Conn_01x04_Male
- added R13: 10k, Resistor_SMD:R_0805_2012Metric, symbol Device:R
- R10: value 1k -> 680
- U4: symbol Interface_CAN_LIN:MCP2515-EST -> jeep-radio-rescue:MCP2515-EST-Interface_CAN_LIN
Connections:
- net labels added: BT_3V3, BT_RESET
- net labels removed: VBAT
- wire segments 169 -> 180
Changed lines of the file:
@@
 Wire Wire Line
 	2700 5050 3050 5050
-Text Label 2850 5050 0    50   ~ 0
-BT_LED
 $Comp
 L Device:Crystal Y1
@@
 XTAL1
 $Comp
-L Interface_CAN_LIN:MCP2515-EST U4
+L jeep-radio-rescue:MCP2515-EST-Interface_CAN_LIN U4
 U 1 1 5B9B70C5
 P 5000 5050
@@
 P 6000 7000
 F 0 "R10" H 6070 7046 50  0000 L CNN
-F 1 "1k" H 6070 6955 50  0000 L CNN
+F 1 "680" H 6070 6955 50  0000 L CNN
 F 2 "Resistor_SMD:R_0805_2012Metric" V 5930 7000 50  0001 C CNN
 F 3 "~" H 6000 7000 50  0001 C CNN
@@
 	6000 6400 6000 6350
 Text Label 6000 6350 0    50   ~ 0
-PWR
+BT_3V3
 Wire Wire Line
 	6000 7150 6000 7350
@@
 	1    0    0    -1
 $EndComp
-Wire Wire Line
-	9350 5100 9200 5100
 $Comp
 L Diode:1N4001 D4
@@
 	0    1    1    0
 $EndComp
-Wire Wire Line
-	9200 5100 9200 5500
 Wire Wire Line
 	8600 5200 8600 5500
@@
 Text Label 2900 1900 0    50   ~ 0
 PWR_9_1
-Text Label 9150 5200 0    50   ~ 0
-VBAT
+Text Label 8700 5200 0    50   ~ 0
+BT_3V3
 Text Label 5700 5650 0    50   ~ 0
 ~RESET~
@@
 Wire Wire Line
 	10250 1500 10250 1550
+Wire Wire Line
+	9200 5000 9350 5000
+Wire Wire Line
+	9200 5000 9200 5500
+$Comp
+L Device:R R13
+U 1 1 5BFF857C
+P 9950 5650
+F 0 "R13" V 9743 5650 50  0000 C CNN
+F 1 "10k" V 9834 5650 50  0000 C CNN
+F 2 "Resistor_SMD:R_0805_2012Metric" V 9880 5650 50  0001 C CNN
+F 3 "~" H 9950 5650 50  0001 C CNN
+	1    9950 5650
+	0    1    1    0
+$EndComp
+Wire Wire Line
+	9350 5300 9350 5650
+Wire Wire Line
+	9350 5650 9800 5650
+Wire Wire Line
+	10100 5650 10550 5650
+Wire Wire Line
+	10550 5650 10550 5200
+Wire Wire Line
+	9350 4800 9100 4800
+Text Label 9100 4800 0    50   ~ 0
+BT_LED
+$Comp
+L power:PWR_FLAG #FLG0104
+U 1 1 5C0302AB
+P 8600 4950
+F 0 "#FLG0104" H 8600 5025 50  0001 C CNN
+F 1 "PWR_FLAG" H 8600 5124 50  0000 C CNN
+F 2 "" H 8600 4950 50  0001 C CNN
+F 3 "~" H 8600 4950 50  0001 C CNN
+	1    8600 4950
+	1    0    0    -1
+$EndComp
+Wire Wire Line
+	8600 4950 8600 5200
+Wire Wire Line
+	10550 5200 10900 5200
+Connection ~ 10550 5200
+Text Label 10650 5200 0    50   ~ 0
+BT_RESET
+$Comp
+L Connector:Conn_01x04_Male J5
+U 1 1 5C063ADC
+P 9950 2750
+F 0 "J5" H 10056 3028 50  0000 C CNN
+F 1 "Conn_01x04_Male" H 10056 2937 50  0000 C CNN
+F 2 "Connector_PinHeader_2.54mm:PinHeader_1x04_P2.54mm_Vertical" H 9950 2750 50  0001 C CNN
+F 3 "~" H 9950 2750 50  0001 C CNN
+	1    9950 2750
+	1    0    0    -1
+$EndComp
+Wire Wire Line
+	10150 2650 10450 2650
+Wire Wire Line
+	10150 2750 10450 2750
+Wire Wire Line
+	10150 2850 10450 2850
+Wire Wire Line
+	10150 2950 10450 2950
+Text Label 10200 2650 0    50   ~ 0
+BT_3V3
+Text Label 10200 2850 0    50   ~ 0
+BT_TX
+Text Label 10200 2750 0    50   ~ 0
+BT_RX
+Text Label 10200 2950 0    50   ~ 0
+BT_RESET
 $EndSCHEMATC
